File: pcb/business-card.sch (KiCad schematic (older format))
At the start: 13 parts, among them J1 HEADER_10, U1 MDBT40, U2 NJM2870, U3 RTF015N03, Y1 Crystal

Commit message: Rename kicad project name to business-card from halakekit_lino
Parts:
- removed BT1: Battery, CR2032_frame:BAT-HLD-001-TRCT, symbol Battery
- removed J1: HEADER_10, simple_headers:Pin_Header_Straight_1x10, symbol HEADER_10
- removed R2: 1K, register_and_condensor:R_0603, symbol R
- removed U3: RTF015N03, mosfet:rtf015n03, symbol RTF015N03
- added J1: Conn_01x06, simple_headers:PinHeader_2x03_P2.00mm_Vertical, symbol Connector_Generic:Conn_01x06
- added J2, J3, J4: Conn_01x01, simple_headers:corner_pad, symbol Connector_Generic:Conn_01x01
- C1, C2, C3, C4, C5: symbol C -> business-card-rescue:C
- R1: symbol R -> business-card-rescue:R
- U1: symbol MDBT40 -> business-card-rescue:MDBT40
- U2: symbol NJM2870 -> business-card-rescue:NJM2870
- Y1: symbol Crystal -> business-card-rescue:Crystal
Connections:
- net labels removed: P4_Drain
- wire segments 29 -> 32
